File: pwr_usb.kicad_sch (KiCad schematic)
At the start: 9 parts, among them J2 USB_C_Receptacle_USB2.0_14P, U3 NCP1117-3.3_SOT223, U4 USBLC6-2P6

Commit message: add subsheets
Parts:
- added C3: 100 nF, symbol Device:C
- added C4: 1000 uF, symbol Device:C_Polarized
- added D1: 1N4728A, Diode_THT:D_DO-41_SOD81_P10.16mm_Horizontal, symbol Diode:1N47xxA
- added J3: Conn_01x02, symbol Connector_Generic:Conn_01x02
- added Q1: Q_NMOS, symbol Device:Q_NMOS
- added R2, R3: 10k, symbol Device:R
Connections:
- net GND: now also C3.2, C4.2, D1.2 (A), Q1.S, R3.2
- net VBUS: now also C3.1
- new net: J3.2 (Pin_2), Q1.D
- new net +6V: C4.1, J3.1 (Pin_1), Q1.G, R2.1
- new net VSENSE: D1.1 (K), R2.2, R3.1
Other:
- note added: "5V -> 3V3"
- note added: "SERVO VIN"
- note added: "USB-C"
- note removed: "Power"
- moved on the sheet: C2, C22, J2, R10, R9, TP1, TP2, U3, U4

Commit message: HELO
Parts:
- C3: footprint (none) -> Capacitor_SMD:C_0402_1005Metric
- C4: footprint (none) -> Capacitor_THT:CP_Radial_D10.0mm_P5.00mm
- J2: footprint (none) -> Connector_USB:USB_C_Receptacle_Molex_105450-0101
- J3: footprint (none) -> Connector_PinHeader_2.54mm:PinHeader_1x02_P2.54mm_Vertical
- R10, R9: footprint (none) -> Resistor_SMD:R_0603_1608Metric
- R2, R3: footprint (none) -> Resistor_SMD:R_0805_2012Metric
- TP1, TP2: footprint (none) -> TestPoint:TestPoint_Plated_Hole_D3.0mm
Changed lines of the file:
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@@
 			)
 		)
-		(property "Footprint" ""
+		(property "Footprint" "Resistor_SMD:R_0603_1608Metric"
 			(at 68.58 38.608 90)
 			(effects
@@
 			)
 		)
-		(property "Footprint" ""
+		(property "Footprint" "TestPoint:TestPoint_Plated_Hole_D3.0mm"
 			(at 85.09 58.42 0)
 			(effects
@@
 			)
 		)
-		(property "Footprint" ""
+		(property "Footprint" "Capacitor_THT:CP_Radial_D10.0mm_P5.00mm"
 			(at 183.8452 38.1 0)
 			(effects
@@
 			)
 		)
-		(property "Footprint" ""
+		(property "Footprint" "Connector_USB:USB_C_Receptacle_Molex_105450-0101"
 			(at 39.37 44.45 0)
 			(effects
@@
 			)
 		)
-		(property "Footprint" ""
+		(property "Footprint" "Resistor_SMD:R_0603_1608Metric"
 			(at 68.58 36.068 90)
 			(effects
@@
 			)
 		)
-		(property "Footprint" ""
+		(property "Footprint" "Resistor_SMD:R_0805_2012Metric"
 			(at 195.072 44.45 90)
 			(effects
@@
 			)
 		)
-		(property "Footprint" ""
+		(property "Footprint" "TestPoint:TestPoint_Plated_Hole_D3.0mm"
 			(at 95.25 50.8 0)
 			(effects
@@
 			)
 		)
-		(property "Footprint" ""
+		(property "Footprint" "Capacitor_SMD:C_0402_1005Metric"
 			(at 98.7552 33.02 0)
 			(effects
@@
 			)
 		)
-		(property "Footprint" ""
+		(property "Footprint" "Connector_PinHeader_2.54mm:PinHeader_1x02_P2.54mm_Vertical"
 			(at 224.79 30.48 0)
 			(effects
@@
 			)
 		)
-		(property "Footprint" ""
+		(property "Footprint" "Resistor_SMD:R_0805_2012Metric"
 			(at 195.072 34.29 90)
 			(effects
