File: spooder_pcb.kicad_pcb (KiCad board)
At the start: 2 copper layers, 42 parts, among them J1 SM03B-SRSS-TB, J11 SM04B-SRSS-TB_LF__SN_, SW3 SW_Push, SW4 SW_Push, U2 RP2350_80QFN, U3 NCP1117-3.3_SOT223, U4 USBLC6-2P6, Y2 ABM8-272-T3

Commit message: HELO
Parts:
- added C10: 100 nF, Capacitor_SMD:C_0402_1005Metric, F.Cu at (209.0, 78.6)
- added C12: 100 nF, Capacitor_SMD:C_0402_1005Metric, F.Cu at (209.0, 80.6)
- added C3: 100 nF, Capacitor_SMD:C_0402_1005Metric, F.Cu at (223.0, 94.5)
- added C4: 1000 uF, Capacitor_THT:CP_Radial_D10.0mm_P5.00mm, F.Cu at (213.5, 83.2)
- added C7: 100 uF, Capacitor_THT:CP_Radial_D5.0mm_P2.00mm, F.Cu at (186.3, 57.0)
- added C8: 100 nF, Capacitor_SMD:C_0402_1005Metric, F.Cu at (209.0, 76.6)
- added C9: 100 uF, Capacitor_THT:CP_Radial_D5.0mm_P2.00mm, F.Cu at (186.3, 63.6)
- added D2: LED, LED_SMD:LED_1206_3216Metric, F.Cu at (204.8, 77.3)
- added D3: LED, LED_SMD:LED_1206_3216Metric, F.Cu at (204.8, 80.7)
- added J10: Conn_01x04_Pin, Connector_PinHeader_2.54mm:PinHeader_1x04_P2.54mm_Vertical, F.Cu at (206.7, 56.0)
- added J12: Conn_01x03_Pin, Connector_PinHeader_2.54mm:PinHeader_1x03_P2.54mm_Vertical, F.Cu at (192.9, 68.3)
- added J13: Conn_01x03_Pin, Connector_PinHeader_2.54mm:PinHeader_1x03_P2.54mm_Vertical, F.Cu at (197.5, 68.3)
- added J14: Conn_01x03_Pin, Connector_PinHeader_2.54mm:PinHeader_1x03_P2.54mm_Vertical, F.Cu at (202.1, 68.3)
- added J15: Conn_01x03_Pin, Connector_PinHeader_2.54mm:PinHeader_1x03_P2.54mm_Vertical, F.Cu at (206.7, 68.3)
- added J16: Conn_01x10_Pin, Connector_PinHeader_2.54mm:PinHeader_1x10_P2.54mm_Vertical, F.Cu at (181.7, 56.0)
- added J17: Conn_01x04_Pin, Connector_PinHeader_2.54mm:PinHeader_1x04_P2.54mm_Vertical, F.Cu at (211.2, 56.0)
- added J18: Conn_01x02_Pin, Connector_PinHeader_2.54mm:PinHeader_1x02_P2.54mm_Vertical, F.Cu at (199.6, 77.9)
- added J2: USB_C_Receptacle_USB2.0_14P, Connector_USB:USB_C_Receptacle_Molex_105450-0101, F.Cu at (218.0, 103.0)
- added J3: Conn_01x02, Connector_PinHeader_2.54mm:PinHeader_1x02_P2.54mm_Vertical, F.Cu at (223.9, 91.2)
- added J7: Conn_01x04_Pin, Connector_PinHeader_2.54mm:PinHeader_1x04_P2.54mm_Vertical, F.Cu at (192.9, 56.0)
- added J8: Conn_01x04_Pin, Connector_PinHeader_2.54mm:PinHeader_1x04_P2.54mm_Vertical, F.Cu at (197.5, 56.0)
- added J9: Conn_01x04_Pin, Connector_PinHeader_2.54mm:PinHeader_1x04_P2.54mm_Vertical, F.Cu at (202.1, 56.0)
- added R10: 5.1k, Resistor_SMD:R_0603_1608Metric, F.Cu at (233.2, 83.0)
- added R2: 10k, Resistor_SMD:R_0805_2012Metric, F.Cu at (233.4, 74.8)
- added R3: 10k, Resistor_SMD:R_0805_2012Metric, F.Cu at (233.4, 77.8)
- added R9: 5.1k, Resistor_SMD:R_0603_1608Metric, F.Cu at (233.2, 80.5)
- added SW1: SW_Push, Button_Switch_SMD:SW_Push_1P1T_NO_Vertical_Wuerth_434133025816, F.Cu at (194.0, 78.0)
- added SW2: SW_Push, Button_Switch_SMD:SW_Push_1P1T_NO_Vertical_Wuerth_434133025816, F.Cu at (194.0, 82.8)
- added TP1: TestPoint, TestPoint:TestPoint_Plated_Hole_D3.0mm, F.Cu at (226.8, 75.0)
- added TP2: TestPoint, TestPoint:TestPoint_Plated_Hole_D3.0mm, F.Cu at (159.6, 54.9)
- C11: footprint Capacitor_THT:C_Radial_D5.0mm_H11.0mm_P2.00mm -> Capacitor_THT:CP_Radial_D5.0mm_P2.00mm
- moved U2 68.6 mm to (132.4, 97.9)
- moved H1 24.3 mm to (149.1, 38.7)
- moved H4 24.3 mm to (149.1, 62.5)
- moved R11 24.3 mm to (164.3, 39.7)
- moved R12 24.3 mm to (164.3, 41.6)
- moved Y2 24.3 mm to (177.0, 46.5)
- moved H2 24.3 mm to (149.1, 46.6)
- moved H3 24.3 mm to (149.1, 54.6)
- moved J11 24.3 mm to (186.8, 38.5)
- moved R1 24.3 mm to (164.3, 35.7)
- moved R13 24.3 mm to (164.3, 43.6)
- moved R5 24.3 mm to (164.3, 37.7)
- moved SW3 24.3 mm to (177.8, 37.1)
- moved SW4 24.3 mm to (177.8, 41.8)
- moved U3 24.3 mm to (167.8, 59.2)
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